File: PCB/HackPad_Neko.kicad_pcb (KiCad board)
At the start: 2 copper layers, 100 x 100 mm, 43 parts, among them J1 Conn_01x04, U1 MOUDLE-SEEEDUINO-XIAO

Commit message: PCB take 2
Parts:
- added R1: 4.7kΩ, Resistor_THT:R_Axial_DIN0204_L3.6mm_D1.6mm_P5.08mm_Horizontal, F.Cu at (204.8, 100.1)
- added R2: 4.7kΩ, Resistor_THT:R_Axial_DIN0204_L3.6mm_D1.6mm_P5.08mm_Horizontal, F.Cu at (208.0, 100.1)
Connections:
- J1 pad 2: +5V -> +3V3
- U1 pad 12: unconnected-(U1-3V3-Pad12) -> +3V3
- U1 pad 14: +5V -> unconnected-(U1-5V-Pad14)
Routing:
- net +3V3: track 0.00 -> 48.7 mm
- net +5V: track 30.4 -> 0.00 mm
- net SDA: track 21.3 -> 35.6 mm
- net SCL: track 17.7 -> 32.0 mm
- net GND: track 30.9 -> 28.9 mm, vias 1 -> 0
- removed copper zone on B.Cu, net GND
