File: PCB/HackPad_Neko.kicad_sch (KiCad schematic)
At the start: 42 parts, among them J1 Conn_01x04, U1 MOUDLE-SEEEDUINO-XIAO

Commit message: PCB take 2
Parts:
- added R1, R2: 4.7kΩ, Resistor_THT:R_Axial_DIN0204_L3.6mm_D1.6mm_P5.08mm_Horizontal, symbol Device:R
Connections:
- net SCL: now also R1.2
- net SDA: now also R2.2
- net +3V3: now reaches U1.12 (3V3)
- net +3V3: now also J1.2 (Pin_2), R1.1, R2.1
- net +5V: no longer names the net of U1.14 (5V)
- net +5V: no longer J1.2 (Pin_2)
